File: Controls.kicad_sch (KiCad schematic)
At the start: 17 parts, among them J1 FOOTSWITCH, J2 JACK CONNECTOR, J3 PCIE_FX, SW1 SW_SPDT, SW2 SW_SPDT, SW3 MINI_SW, SW4 MINI_SW

Commit message: Minor changes
Updated some elements in the silkscreen layer.
Neeed to remove some components from the paste layer.
Parts:
- H1: footprint Mounting_Wuerth:Mounting_Wuerth_WA-SMSI-M2_H1.5mm_9774015243 -> Mounting_Wuerth:Mounting_Wuerth_WA-SMSI-M2.5_H1.5mm_9774015151
Changed lines of the file:
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@@
 			)
 		)
-		(property "Footprint" "Mounting_Wuerth:Mounting_Wuerth_WA-SMSI-M2_H1.5mm_9774015243"
+		(property "Footprint" "Mounting_Wuerth:Mounting_Wuerth_WA-SMSI-M2.5_H1.5mm_9774015151"
 			(at 80.01 170.18 0)
 			(hide yes)
