File: EffectsBase.kicad_pcb (KiCad board)
At the start: 2 copper layers, 59 x 98 mm, 36 parts, among them J1 FOOTSWITCH, J2 JACK CONNECTOR, J3 PCIE_FX, Q1 SI2301BDS, SW1 SW_SPDT, SW2 SW_SPDT, SW3 MINI_SW, SW4 MINI_SW, U1 ICL7660S

Commit message: Minor changes
Updated some elements in the silkscreen layer.
Neeed to remove some components from the paste layer.
Parts:
- added REF**: MT, Logos:MT, F.Cu at (172.0, 65.8)
- H1: footprint Mounting_Wuerth:Mounting_Wuerth_WA-SMSI-M2_H1.5mm_9774015243 -> Mounting_Wuerth:Mounting_Wuerth_WA-SMSI-M2.5_H1.5mm_9774015151
- moved J1 0.07 mm to (150.0, 135.4)
Other:
- board text added: "DAVID MT"
- board text added: "EFFECTS BASE"
- board text added: "PD 08/26"
- board text added: "V1.0 REV A"
