File: Power.kicad_sch (KiCad schematic)
At the start: 18 parts, among them Q1 SI2301BDS, U1 ICL7660S

Commit message: Minor changes
Updated some elements in the silkscreen layer.
Neeed to remove some components from the paste layer.
Parts:
- R1: value 100 -> 10
Changed lines of the file:
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@@
 			)
 		)
-		(property "Value" "100"
+		(property "Value" "10"
 			(at 96.52 113.0299 0)
 			(show_name no)
